Commit message: changed the /dev/ttyUSB0 to /tmp/ttyUR and disconnected the tool_communication from the standard ur_robotiq_control.launch.py launchfile

File: robotiq_description/urdf/2f_140.ros2_control.xacro (robot description, xacro)
@@ -10,5 +10,5 @@
         use_fake_hardware:=false
         fake_sensor_commands:=false
-        com_port:=/dev/ttyUSB0">
+        com_port:=/tmp/ttyUR">
         <ros2_control name="${name}" type="system">
             <!-- Plugins -->
@@ -73,6 +73,6 @@
                     </xacro:unless>
                 </joint>
-                <joint name="${prefix}right_inner_knuckle_joint">
-                    <param name="mimic">${prefix}finger_joint</param>
+                <joint name="${prefix}robotiq_140_left_finger_tip_joint">
+                    <param name="mimic">${prefix}robotiq_140_left_knuckle_joint</param>
                     <param name="multiplier">-1</param>
                     <xacro:unless value="${sim_ignition}">
@@ -82,6 +82,6 @@
                     </xacro:unless>
                 </joint>
-                <joint name="${prefix}right_inner_finger_joint">
-                    <param name="mimic">${prefix}finger_joint</param>
+                <joint name="${prefix}robotiq_140_right_finger_tip_joint">
+                    <param name="mimic">${prefix}robotiq_140_left_knuckle_joint</param>
                     <param name="multiplier">1</param>
                     <xacro:unless value="${sim_ignition}">

File: robotiq_description/urdf/robotiq_2f_140_macro.urdf.xacro (robot description, xacro)
@@ -13,5 +13,5 @@
         fake_sensor_commands:=false
         include_ros2_control:=true
-        com_port:=/dev/ttyUSB0">
+        com_port:=/tmp/ttyUR">
         <!-- ros2 control include -->
         <xacro:include filename="$(find robotiq_description)/urdf/2f_140.ros2_control.xacro" />
